File: shimu.kicad_pcb (KiCad board)
At the start: 4 copper layers, 26.7 x 20.3 mm, 24 parts, among them J1 Conn_01x06_Pin, J2 Conn_01x04_Pin, U1 TLV75533PDRV, U2 ICM-45686

Commit message: PCB Rev B: improved ground via placement
Routing:
- net GND: vias 46 -> 52
Other:
- board text added: "Rev. B"
- board text removed: "Rev. A"
